Commit message: alterações no tamanho/peso

File: install/laser_rahcm_visualization/share/laser_rahcm_visualization/urdf/arm.urdf.xacro (robot description, xacro)
@@ -17,9 +17,9 @@
       <inertial>
         <origin xyz="0 0 0.55" rpy="0 0 0"/>
-        <mass value="12.5"/>
+        <mass value="10"/>
         <inertia
-          ixx="${(1.0/12.0) * 12.5 * (3*(0.1*0.1) + 1.1*1.1)}"
-          iyy="${(1.0/12.0) * 12.5 * (3*(0.1*0.1) + 1.1*1.1)}"
-          izz="${(1.0/2.0) * 12.5 * (0.1*0.1)}"
+          ixx="${(1.0/12.0) * 10.0 * (3*(0.1*0.1) + 1.1*1.1)}"
+          iyy="${(1.0/12.0) * 10.0 * (3*(0.1*0.1) + 1.1*1.1)}"
+          izz="${(1.0/2.0) * 10.0 * (0.1*0.1)}"
           ixy="0.0" ixz="0.0" iyz="0.0"/>
       </inertial>

File: install/laser_rahcm_visualization/share/laser_rahcm_visualization/urdf/base.urdf.xacro (robot description, xacro)
@@ -6,5 +6,5 @@
       <visual>
         <geometry>
-          <box size="0.8 1.5 0.6"/>
+          <box size="0.8 1 0.6"/>
         </geometry>
         <material name="gray"/>
@@ -17,9 +17,9 @@
       <inertial>
         <origin xyz="0 0 0.3" rpy="0 0 0"/>
-        <mass value="80"/>
+        <mass value="90"/>
         <inertia
-          ixx="${1.5/12.0 * 80.0 * (0.8*0.8 + 0.6*0.6)}"
-          iyy="${1.5/12.0 * 80.0 * (1.5*1.5 + 0.6*0.6)}"
-          izz="${1.5/12.0 * 80.0 * (0.8*0.8 + 1.5*1.5)}"
+          ixx="${1.0/12.0 * 90.0 * (0.8*0.8 + 0.6*0.6)}"
+          iyy="${1.0/12.0 * 90.0 * (1.0*1.0 + 0.6*0.6)}"
+          izz="${1.0/12.0 * 90.0 * (0.8*0.8 + 1.0*1.0)}"
           ixy="0.0" ixz="0.0" iyz="0.0"/>
       </inertial>

File: install/laser_rahcm_visualization/share/laser_rahcm_visualization/urdf/rahcm.urdf.xacro (robot description, xacro)
@@ -15,11 +15,11 @@
   <xacro:base name="base"/>
   <!-- Braços e Rodas -->
-  <xacro:arm name="arm_front_left" parent="base_link" xyz="-0.65 0.45 -0.3" rpy="0 0.6 0"/>
+  <xacro:arm name="arm_front_left" parent="base_link" xyz="-0.65 0.35 -0.3" rpy="0 0.6 0"/>
   <xacro:wheel name="wheel_front_left" parent="arm_front_left" xyz="0 0 -0.3" rpy="0 0 0"/>
-  <xacro:arm name="arm_front_right" parent="base_link" xyz="-0.65 -0.45 -0.3" rpy="0 0.6 0"/>
+  <xacro:arm name="arm_front_right" parent="base_link" xyz="-0.65 -0.35 -0.3" rpy="0 0.6 0"/>
   <xacro:wheel name="wheel_front_right" parent="arm_front_right" xyz="0 0 -0.3" rpy="0 0 0"/>
-  <xacro:arm name="arm_rear_left" parent="base_link" xyz="0.65 0.45 -0.3" rpy="0 -0.6 0"/>
+  <xacro:arm name="arm_rear_left" parent="base_link" xyz="0.65 0.35 -0.3" rpy="0 -0.6 0"/>
   <xacro:wheel name="wheel_rear_left" parent="arm_rear_left" xyz="0 0 -0.3" rpy="0 0 0"/>
-  <xacro:arm name="arm_rear_right" parent="base_link" xyz="0.65 -0.45 -0.3" rpy="0 -0.6 0"/>
+  <xacro:arm name="arm_rear_right" parent="base_link" xyz="0.65 -0.35 -0.3" rpy="0 -0.6 0"/>
   <xacro:wheel name="wheel_rear_right" parent="arm_rear_right" xyz="0 0 -0.3" rpy="0 0 0"/>
   <gazebo>

File: install/laser_rahcm_visualization/share/laser_rahcm_visualization/urdf/wheel.urdf.xacro (robot description, xacro)
@@ -1,25 +1,25 @@
 <?xml version="1.0"?>
 <robot xmlns:xacro="http://ros.org/wiki/xacro">
-  <!-- Braço do robô -->
-   <xacro:macro name="arm" params="name parent xyz rpy">
+  <!-- Roda do robô -->
+  <xacro:macro name="wheel" params="name parent xyz rpy">
     <link name="${name}">
       <visual>
         <geometry>
-          <cylinder length="1.1" radius="0.1"/>
+          <sphere radius="0.3"/>
         </geometry>
-        <material name="gray"/>
+        <material name="black"/>
       </visual>
       <collision>
         <geometry>
-          <cylinder length="1.1" radius="0.1"/>
+          <sphere radius="0.3"/>
         </geometry>
       </collision>
       <inertial>
-        <origin xyz="0 0 0.55" rpy="0 0 0"/>
-        <mass value="12.5"/>
+        <origin xyz="0 0 0" rpy="0 0 0"/>
+        <mass value="5"/>
         <inertia
-          ixx="${(1.0/12.0) * 12.5 * (3*(0.1*0.1) + 1.1*1.1)}"
-          iyy="${(1.0/12.0) * 12.5 * (3*(0.1*0.1) + 1.1*1.1)}"
-          izz="${(1.0/2.0) * 12.5 * (0.1*0.1)}"
+          ixx="${(2/5) * 5.0 * (0.3*0.3)}"
+          iyy="${(2/5) * 5.0 * (0.3*0.3)}"
+          izz="${(2/5) * 5.0 * (0.3*0.3)}"
           ixy="0.0" ixz="0.0" iyz="0.0"/>
       </inertial>
