Commit message: adição da modelagem da roda como elemento visual e correção de colisões e inercias do modelo

File: urdf/rahcm.urdf.xacro (robot description, xacro)
@@ -5,4 +5,5 @@
   <xacro:include filename="arm.urdf.xacro"/>
   <xacro:include filename="wheel.urdf.xacro"/>
+  <xacro:include filename="wheel_arm_joint.urdf.xacro"/>
   <!-- Define materiais -->
   <material name="gray">
@@ -16,13 +17,14 @@
   <!-- Braços e Rodas -->
   <xacro:arm name="arm_front_left" parent="base_link" xyz="-0.65 0.45 -0.3" rpy="0 0.6 0"/>
-  <xacro:wheel name="wheel_front_left" parent="arm_front_left" xyz="0 0 -0.3" rpy="0 0 0"/>
+  <xacro:joint_arm name="joint_arm_front_left" parent="arm_front_left" xyz="0 0 -0.5" rpy="0 1 0"/>
+  <xacro:wheel name="wheel_front_left" parent="joint_arm_front_left" xyz="0 0 -0.25" rpy="0 0 0"/>
   <xacro:arm name="arm_front_right" parent="base_link" xyz="-0.65 -0.45 -0.3" rpy="0 0.6 0"/>
-  <xacro:wheel name="wheel_front_right" parent="arm_front_right" xyz="0 0 -0.3" rpy="0 0 0"/>
+  <xacro:joint_arm name="joint_arm_front_right" parent="arm_front_right" xyz="0 0 -0.5" rpy="0 1 0"/>
+  <xacro:wheel name="wheel_front_right" parent="joint_arm_front_right" xyz="0 0 -0.25" rpy="0 0 0"/>
   <xacro:arm name="arm_rear_left" parent="base_link" xyz="0.65 0.45 -0.3" rpy="0 -0.6 0"/>
-  <xacro:wheel name="wheel_rear_left" parent="arm_rear_left" xyz="0 0 -0.3" rpy="0 0 0"/>
+  <xacro:joint_arm name="joint_arm_rear_left" parent="arm_rear_left" xyz="0 0 -0.5" rpy="0 -1 0"/>
+  <xacro:wheel name="wheel_rear_left" parent="joint_arm_rear_left" xyz="0 0 -0.25" rpy="0 0 0"/>
   <xacro:arm name="arm_rear_right" parent="base_link" xyz="0.65 -0.45 -0.3" rpy="0 -0.6 0"/>
-  <xacro:wheel name="wheel_rear_right" parent="arm_rear_right" xyz="0 0 -0.3" rpy="0 0 0"/>
-  <gazebo>
-    <static>false</static>
-  </gazebo>
+  <xacro:joint_arm name="joint_arm_rear_right" parent="arm_rear_right" xyz="0 0 -0.5" rpy="0 -1 0"/>
+  <xacro:wheel name="wheel_rear_right" parent="joint_arm_rear_right" xyz="0 0 -0.25" rpy="0 0 0"/>
 </robot>

File: urdf/wheel.urdf.xacro (robot description, xacro)
@@ -1,16 +1,17 @@
 <?xml version="1.0"?>
 <robot xmlns:xacro="http://ros.org/wiki/xacro">
-  <!-- Roda do robô -->
+  <!-- Roda do robô  -->
   <xacro:macro name="wheel" params="name parent xyz rpy">
+    <!-- Link da roda -->
     <link name="${name}">
       <visual>
         <geometry>
-          <sphere radius="0.3"/>
+          <mesh filename="package://laser_rahcm_visualization/meshes/wheel.stl" scale="0.01 0.01 0.01"/>
         </geometry>
-        <material name="black"/>
+        <material name="gray"/>
       </visual>
       <collision>
         <geometry>
-          <sphere radius="0.3"/>
+          <cylinder radius="0.3" length="0.3"/>
         </geometry>
       </collision>
@@ -19,7 +20,7 @@
         <mass value="10"/>
         <inertia
-          ixx="${(2/5) * 10.0 * (0.3*0.3)}"
-          iyy="${(2/5) * 10.0 * (0.3*0.3)}"
-          izz="${(2/5) * 10.0 * (0.3*0.3)}"
+          ixx="${(1.0/12.0) * 10.0 * (3*(0.3*0.3) + 0.3*0.3)}"
+          iyy="${(1.0/12.0) * 10.0 * (3*(0.3*0.3) + 0.3*0.3)}"
+          izz="${(1.0/2.0) * 10.0 * (0.3*0.3)}"
           ixy="0.0" ixz="0.0" iyz="0.0"/>
       </inertial>
@@ -27,8 +28,8 @@
     <joint name="joint_${name}" type="continuous">
       <parent link="${parent}"/>
-      <child link="${name}"/>
+      <child  link="${name}"/>
       <origin xyz="${xyz}" rpy="${rpy}"/>
-      <axis xyz="1 0 0"/>
-      <limit effort="5.0" velocity="10.0"/>
+      <axis  xyz="0 0 1"/>
+      <limit  effort="5.0" velocity="10.0"/>
       <dynamics damping="0.1" friction="0.1"/>
     </joint>
