Commit message: alterações nas rodas e estão funcionando como o esperado

File: urdf/wheel.urdf.xacro (robot description, xacro)
@@ -25,5 +25,5 @@
       </inertial>
     </link>
-    <joint name="joint_${name}" type="revolute">
+    <joint name="joint_${name}" type="continuous">
       <parent link="${parent}"/>
       <child link="${name}"/>

Commit message: mudança na imagem

File: urdf/wheel.urdf.xacro (robot description, xacro)
@@ -7,5 +7,5 @@
       <visual>
         <geometry>
-          <mesh filename="package://laser_rahcm_visualization/meshes/wheel.stl" scale="0.01 0.01 0.01"/>
+          <mesh filename="package://laser_rahcm_visualization/meshes/wheel.dae" scale="0.01 0.01 0.01"/>
         </geometry>
         <material name="gray"/>
