Commit message: adição da modelagem dos braços e modificação na posição dos braços

File: urdf/arm.urdf.xacro (robot description, xacro)
@@ -5,6 +5,7 @@
     <link name="${name}">
       <visual>
+        <origin xyz="0 0 -0.5" rpy="0 -0.4 0"/>
         <geometry>
-          <cylinder length="1.1" radius="0.1"/>
+          <mesh filename="package://laser_rahcm_visualization/meshes/arm.stl" scale="0.018 0.018 0.018"/>
         </geometry>
         <material name="gray"/>

File: urdf/rahcm.urdf.xacro (robot description, xacro)
@@ -16,9 +16,9 @@
   <xacro:base name="base"/>
   <!-- Braços e Rodas -->
-  <xacro:arm name="arm_front_left" parent="base_link" xyz="-0.65 0.45 -0.3" rpy="0 0.6 0"/>
-  <xacro:joint_arm name="joint_arm_front_left" parent="arm_front_left" xyz="0 0 -0.5" rpy="0 1 0"/>
+  <xacro:arm name="arm_front_left" parent="base_link" xyz="-0.65 0.45 -0.3" rpy="0 -0.6 3.14"/>
+  <xacro:joint_arm name="joint_arm_front_left" parent="arm_front_left" xyz="0 0 -0.5" rpy="0 -1 0"/>
   <xacro:wheel name="wheel_front_left" parent="joint_arm_front_left" xyz="0 0 -0.25" rpy="0 0 0"/>
-  <xacro:arm name="arm_front_right" parent="base_link" xyz="-0.65 -0.45 -0.3" rpy="0 0.6 0"/>
-  <xacro:joint_arm name="joint_arm_front_right" parent="arm_front_right" xyz="0 0 -0.5" rpy="0 1 0"/>
+  <xacro:arm name="arm_front_right" parent="base_link" xyz="-0.65 -0.45 -0.3" rpy="0 -0.6 3.14"/>
+  <xacro:joint_arm name="joint_arm_front_right" parent="arm_front_right" xyz="0 0 -0.5" rpy="0 -1 0"/>
   <xacro:wheel name="wheel_front_right" parent="joint_arm_front_right" xyz="0 0 -0.25" rpy="0 0 0"/>
   <xacro:arm name="arm_rear_left" parent="base_link" xyz="0.65 0.45 -0.3" rpy="0 -0.6 0"/>

File: urdf/wheel.urdf.xacro (robot description, xacro)
@@ -6,4 +6,5 @@
     <link name="${name}">
       <visual>
+        <origin xyz="0 0 0" rpy="0 0 0"/>
         <geometry>
           <mesh filename="package://laser_rahcm_visualization/meshes/wheel.dae" scale="0.01 0.01 0.01"/>

Commit message: modelo visual final, atualização no tamanho, colisoões e inercias com modelagens como elemento visual

File: urdf/arm.urdf.xacro (robot description, xacro)
@@ -5,22 +5,22 @@
     <link name="${name}">
       <visual>
-        <origin xyz="0 0 -0.5" rpy="0 -0.4 0"/>
+        <origin xyz="0 0 -0.3" rpy="0 -0.4 0"/>
         <geometry>
-          <mesh filename="package://laser_rahcm_visualization/meshes/arm.stl" scale="0.018 0.018 0.018"/>
+          <mesh filename="package://laser_rahcm_visualization/meshes/arm.stl" scale="0.01 0.01 0.011"/>
         </geometry>
-        <material name="gray"/>
+        <material name="green"/>
       </visual>
       <collision>
         <geometry>
-          <cylinder length="1.1" radius="0.1"/>
+          <cylinder length="0.55" radius="0.05"/>
         </geometry>
       </collision>
       <inertial>
-        <origin xyz="0 0 0.55" rpy="0 0 0"/>
+        <origin xyz="0 0 0" rpy="0 0 0"/>
         <mass value="12.5"/>
         <inertia
-          ixx="${(1.0/12.0) * 12.5 * (3*(0.1*0.1) + 1.1*1.1)}"
-          iyy="${(1.0/12.0) * 12.5 * (3*(0.1*0.1) + 1.1*1.1)}"
-          izz="${(1.0/2.0) * 12.5 * (0.1*0.1)}"
+          ixx="${(1.0/12.0) * 12.5 * (3*(0.05*0.05) + 0.55*0.55)}"
+          iyy="${(1.0/12.0) * 12.5 * (3*(0.05*0.05) + 0.55*0.55)}"
+          izz="${(1.0/2.0) * 12.5 * (0.05*0.05)}"
           ixy="0.0" ixz="0.0" iyz="0.0"/>
       </inertial>

File: urdf/base.urdf.xacro (robot description, xacro)
@@ -5,21 +5,22 @@
     <link name="base_link">
       <visual>
+      <origin xyz="0 0 -0.5" rpy="0 0 0"/>
         <geometry>
-          <box size="0.8 1.5 0.6"/>
+          <mesh filename="package://laser_rahcm_visualization/meshes/chassi.dae" scale="0.0113 0.011 0.0125"/>
         </geometry>
-        <material name="gray"/>
+        <material name="white"/>
       </visual>
       <collision>
         <geometry>
-          <box size="0.8 1.5 0.6"/>
+          <box size="0.8 1.1 0.6"/>
         </geometry>
       </collision>
       <inertial>
-        <origin xyz="0 0 0.3" rpy="0 0 0"/>
-        <mass value="60"/>
+        <origin xyz="0 0 0" rpy="0 0 0"/>
+        <mass value="50"/>
         <inertia
-          ixx="${1.5/12.0 * 60.0 * (0.8*0.8 + 0.6*0.6)}"
-          iyy="${1.5/12.0 * 60.0 * (1.5*1.5 + 0.6*0.6)}"
-          izz="${1.5/12.0 * 60.0 * (0.8*0.8 + 1.5*1.5)}"
+          ixx="${1.1/12.0 * 50.0 * (0.8*0.8 + 0.6*0.6)}"
+          iyy="${1.1/12.0 * 50.0 * (1.1*1.1 + 0.6*0.6)}"
+          izz="${1.1/12.0 * 50.0 * (0.8*0.8 + 1.1*1.1)}"
           ixy="0.0" ixz="0.0" iyz="0.0"/>
       </inertial>

File: urdf/rahcm.urdf.xacro (robot description, xacro)
@@ -13,18 +13,24 @@
     <color rgba="0.0 0.0 0.0 1.0"/>
   </material>
+  <material name="green">
+    <color rgba="0.0 0.8 0.0 1.0"/>
+  </material>
+  <material name="white">
+    <color rgba="1.0 1.0 1.0 1.0"/>
+  </material>
   <!-- Corpo principal -->
   <xacro:base name="base"/>
   <!-- Braços e Rodas -->
-  <xacro:arm name="arm_front_left" parent="base_link" xyz="-0.65 0.45 -0.3" rpy="0 -0.6 3.14"/>
-  <xacro:joint_arm name="joint_arm_front_left" parent="arm_front_left" xyz="0 0 -0.5" rpy="0 -1 0"/>
+  <xacro:arm name="arm_front_left" parent="base_link" xyz="-0.45 0.4 -0.3" rpy="0 -0.9 3.14"/>
+  <xacro:joint_arm name="joint_arm_front_left" parent="arm_front_left" xyz="0 0 -0.35" rpy="0 -0.7 0"/>
   <xacro:wheel name="wheel_front_left" parent="joint_arm_front_left" xyz="0 0 -0.25" rpy="0 0 0"/>
-  <xacro:arm name="arm_front_right" parent="base_link" xyz="-0.65 -0.45 -0.3" rpy="0 -0.6 3.14"/>
-  <xacro:joint_arm name="joint_arm_front_right" parent="arm_front_right" xyz="0 0 -0.5" rpy="0 -1 0"/>
+  <xacro:arm name="arm_front_right" parent="base_link" xyz="-0.45 -0.38 -0.3" rpy="0 -0.9 3.14"/>
+  <xacro:joint_arm name="joint_arm_front_right" parent="arm_front_right" xyz="0 0 -0.35" rpy="0 -0.7 0"/>
   <xacro:wheel name="wheel_front_right" parent="joint_arm_front_right" xyz="0 0 -0.25" rpy="0 0 0"/>
-  <xacro:arm name="arm_rear_left" parent="base_link" xyz="0.65 0.45 -0.3" rpy="0 -0.6 0"/>
-  <xacro:joint_arm name="joint_arm_rear_left" parent="arm_rear_left" xyz="0 0 -0.5" rpy="0 -1 0"/>
+  <xacro:arm name="arm_rear_left" parent="base_link" xyz="0.45 0.4 -0.3" rpy="0 -0.9 0"/>
+  <xacro:joint_arm name="joint_arm_rear_left" parent="arm_rear_left" xyz="0 0 -0.35" rpy="0 -0.7 0"/>
   <xacro:wheel name="wheel_rear_left" parent="joint_arm_rear_left" xyz="0 0 -0.25" rpy="0 0 0"/>
-  <xacro:arm name="arm_rear_right" parent="base_link" xyz="0.65 -0.45 -0.3" rpy="0 -0.6 0"/>
-  <xacro:joint_arm name="joint_arm_rear_right" parent="arm_rear_right" xyz="0 0 -0.5" rpy="0 -1 0"/>
+  <xacro:arm name="arm_rear_right" parent="base_link" xyz="0.45 -0.38 -0.3" rpy="0 -0.9 0"/>
+  <xacro:joint_arm name="joint_arm_rear_right" parent="arm_rear_right" xyz="0 0 -0.35" rpy="0 -0.7 0"/>
   <xacro:wheel name="wheel_rear_right" parent="joint_arm_rear_right" xyz="0 0 -0.25" rpy="0 0 0"/>
 </robot>

File: urdf/wheel.urdf.xacro (robot description, xacro)
@@ -8,5 +8,5 @@
         <origin xyz="0 0 0" rpy="0 0 0"/>
         <geometry>
-          <mesh filename="package://laser_rahcm_visualization/meshes/wheel.dae" scale="0.01 0.01 0.01"/>
+          <mesh filename="package://laser_rahcm_visualization/meshes/wheel.dae" scale="0.01 0.01 0.013"/>
         </geometry>
         <material name="gray"/>
@@ -14,14 +14,14 @@
       <collision>
         <geometry>
-          <cylinder radius="0.3" length="0.3"/>
+          <cylinder radius="0.3" length="0.55"/>
         </geometry>
       </collision>
       <inertial>
         <origin xyz="0 0 0" rpy="0 0 0"/>
-        <mass value="10"/>
+        <mass value="12.5"/>
         <inertia
-          ixx="${(1.0/12.0) * 10.0 * (3*(0.3*0.3) + 0.3*0.3)}"
-          iyy="${(1.0/12.0) * 10.0 * (3*(0.3*0.3) + 0.3*0.3)}"
-          izz="${(1.0/2.0) * 10.0 * (0.3*0.3)}"
+          ixx="${(1.0/12.0) * 12.5 * (3*(0.3*0.3) + 0.55*0.55)}"
+          iyy="${(1.0/12.0) * 12.5 * (3*(0.3*0.3) + 0.55*0.55)}"
+          izz="${(1.0/2.0) * 12.5 * (0.3*0.3)}"
           ixy="0.0" ixz="0.0" iyz="0.0"/>
       </inertial>

File: urdf/wheel_arm_joint.urdf.xacro (robot description, xacro)
@@ -6,5 +6,5 @@
       <visual>
         <geometry>
-          <cylinder length="0.25" radius="0.1"/>
+          <cylinder length="0.23" radius="0.04"/>
         </geometry>
         <material name="gray"/>
@@ -12,5 +12,5 @@
       <collision>
         <geometry>
-          <cylinder length="0.25" radius="0.1"/>
+          <cylinder length="0.23" radius="0.04"/>
         </geometry>
       </collision>
@@ -19,7 +19,7 @@
         <mass value="2.0"/>
         <inertia
-          ixx="${(1.0/12.0) * 2.0 * (3*(0.1*0.1) + 0.2*0.2)}"
-          iyy="${(1.0/12.0) * 2.0 * (3*(0.1*0.1) + 0.2*0.2)}"
-          izz="${(1.0/2.0) * 2.0 * (0.1*0.1)}"
+          ixx="${(1.0/12.0) * 2.0 * (3*(0.04*0.04) + 0.23*0.23)}"
+          iyy="${(1.0/12.0) * 2.0 * (3*(0.04*0.04) + 0.23*0.23)}"
+          izz="${(1.0/2.0) * 2.0 * (0.04*0.04)}"
           ixy="0.0" ixz="0.0" iyz="0.0"/>
       </inertial>

Commit message: alterações solicitadas por gabriel

File: urdf/arm.urdf.xacro (robot description, xacro)
@@ -5,11 +5,12 @@
     <link name="${name}">
       <visual>
-        <origin xyz="0 0 -0.3" rpy="0 -0.4 0"/>
+        <origin xyz="0.1 0 -0.6" rpy="0 -0.6 0"/>
         <geometry>
-          <mesh filename="package://laser_rahcm_visualization/meshes/arm.stl" scale="0.01 0.01 0.011"/>
+          <mesh filename="package://laser_rahcm_visualization/meshes/arm.stl" scale="0.01 0.01 0.012"/>
         </geometry>
         <material name="green"/>
       </visual>
       <collision>
+        <origin xyz="0 0 -0.3" rpy="0 -0.4 0"/>
         <geometry>
           <cylinder length="0.55" radius="0.05"/>
@@ -17,17 +18,20 @@
       </collision>
       <inertial>
-        <origin xyz="0 0 0" rpy="0 0 0"/>
-        <mass value="12.5"/>
+        <origin xyz="0 0 -0.3" rpy="0 -0.4 0"/>
+        <mass value="3.0"/>
         <inertia
-          ixx="${(1.0/12.0) * 12.5 * (3*(0.05*0.05) + 0.55*0.55)}"
-          iyy="${(1.0/12.0) * 12.5 * (3*(0.05*0.05) + 0.55*0.55)}"
-          izz="${(1.0/2.0) * 12.5 * (0.05*0.05)}"
+          ixx="${(1.0/2.0) * 3.0 * (0.55*0.55)}"
+          iyy="${(1.0/12.0) * 3.0 * (3*(0.05*0.05) + 0.55*0.55)}"
+          izz="${(1.0/12.0) * 3.0 * (3*(0.05*0.05) + 0.55*0.55)}"
           ixy="0.0" ixz="0.0" iyz="0.0"/>
       </inertial>
     </link>
-    <joint name="joint_${name}" type="fixed">
+    <joint name="joint_base_${name}" type="fixed">
       <parent link="${parent}"/>
       <child link="${name}"/>
       <origin xyz="${xyz}" rpy="${rpy}"/>
+      <axis xyz="0 1 0"/>
+      <limit effort="10.0" velocity="1.0" lower="-0.2" upper="0.4"/>
+      <dynamics damping="5.0" friction="5.0"/>
     </joint>
   </xacro:macro>

File: urdf/base.urdf.xacro (robot description, xacro)
@@ -5,22 +5,23 @@
     <link name="base_link">
       <visual>
-      <origin xyz="0 0 -0.5" rpy="0 0 0"/>
+      <origin xyz="-0.001 0 -0.8" rpy="0 0 0"/>
         <geometry>
-          <mesh filename="package://laser_rahcm_visualization/meshes/chassi.dae" scale="0.0113 0.011 0.0125"/>
+          <mesh filename="package://laser_rahcm_visualization/meshes/chassi.dae" scale="0.0115 0.011 0.0095"/>
         </geometry>
         <material name="white"/>
       </visual>
       <collision>
+        <origin xyz="0 0 -0.5" rpy="0 0 0"/>
         <geometry>
-          <box size="0.8 1.1 0.6"/>
+          <box size="0.71 1.35 0.55"/>
         </geometry>
       </collision>
       <inertial>
-        <origin xyz="0 0 0" rpy="0 0 0"/>
-        <mass value="50"/>
+        <origin xyz="0 0 -0.5" rpy="0 0 0"/>
+        <mass value="10.0"/>
         <inertia
-          ixx="${1.1/12.0 * 50.0 * (0.8*0.8 + 0.6*0.6)}"
-          iyy="${1.1/12.0 * 50.0 * (1.1*1.1 + 0.6*0.6)}"
-          izz="${1.1/12.0 * 50.0 * (0.8*0.8 + 1.1*1.1)}"
+          ixx="${1.0/12.0 * 10.0 * (1.2*1.2 + 0.5*0.5)}"
+          iyy="${1.0/12.0 * 10.0 * (0.8*0.8 + 0.5*0.5)}"
+          izz="${1.0/12.0 * 10.0 * (0.8*0.8 + 1.1*1.1)}"
           ixy="0.0" ixz="0.0" iyz="0.0"/>
       </inertial>

File: urdf/rahcm.urdf.xacro (robot description, xacro)
@@ -1,9 +1,10 @@
 <?xml version="1.0"?>
 <robot name="laser_rahcm_visualization" xmlns:xacro="http://ros.org/wiki/xacro">
-  <!-- Importa os módulos -->
   <xacro:include filename="base.urdf.xacro"/>
   <xacro:include filename="arm.urdf.xacro"/>
+  <xacro:include filename="wheel_arm_joint.urdf.xacro"/>
   <xacro:include filename="wheel.urdf.xacro"/>
-  <xacro:include filename="wheel_arm_joint.urdf.xacro"/>
+  <xacro:property name="controller_config_path"
+                  value="$(find laser_rahcm_visualization)/config/rahcm_controllers.yaml" />
   <!-- Define materiais -->
   <material name="gray">
@@ -19,18 +20,97 @@
     <color rgba="1.0 1.0 1.0 1.0"/>
   </material>
-  <!-- Corpo principal -->
   <xacro:base name="base"/>
-  <!-- Braços e Rodas -->
-  <xacro:arm name="arm_front_left" parent="base_link" xyz="-0.45 0.4 -0.3" rpy="0 -0.9 3.14"/>
-  <xacro:joint_arm name="joint_arm_front_left" parent="arm_front_left" xyz="0 0 -0.35" rpy="0 -0.7 0"/>
-  <xacro:wheel name="wheel_front_left" parent="joint_arm_front_left" xyz="0 0 -0.25" rpy="0 0 0"/>
-  <xacro:arm name="arm_front_right" parent="base_link" xyz="-0.45 -0.38 -0.3" rpy="0 -0.9 3.14"/>
-  <xacro:joint_arm name="joint_arm_front_right" parent="arm_front_right" xyz="0 0 -0.35" rpy="0 -0.7 0"/>
-  <xacro:wheel name="wheel_front_right" parent="joint_arm_front_right" xyz="0 0 -0.25" rpy="0 0 0"/>
-  <xacro:arm name="arm_rear_left" parent="base_link" xyz="0.45 0.4 -0.3" rpy="0 -0.9 0"/>
-  <xacro:joint_arm name="joint_arm_rear_left" parent="arm_rear_left" xyz="0 0 -0.35" rpy="0 -0.7 0"/>
-  <xacro:wheel name="wheel_rear_left" parent="joint_arm_rear_left" xyz="0 0 -0.25" rpy="0 0 0"/>
-  <xacro:arm name="arm_rear_right" parent="base_link" xyz="0.45 -0.38 -0.3" rpy="0 -0.9 0"/>
-  <xacro:joint_arm name="joint_arm_rear_right" parent="arm_rear_right" xyz="0 0 -0.35" rpy="0 -0.7 0"/>
-  <xacro:wheel name="wheel_rear_right" parent="joint_arm_rear_right" xyz="0 0 -0.25" rpy="0 0 0"/>
+  <xacro:arm name="arm_rear_right" parent="base_link" xyz="-0.4 0.4 -0.4" rpy="0 -0.9 3.14"/>
+  <xacro:joint_arm name="arm_joint_wheel_rear_right" parent="arm_rear_right" xyz="0.16 0 -0.68" rpy="0 -0.9 3.14"/>
+  <xacro:wheel name="wheel_rear_right" parent="arm_joint_wheel_rear_right" xyz="-0.25 0 0" rpy="0 0 0"/>
+  <xacro:arm name="arm_front_right" parent="base_link" xyz="-0.4 -0.38 -0.4" rpy="0 -0.9 3.14"/>
+  <xacro:joint_arm name="arm_joint_wheel_front_right" parent="arm_front_right" xyz="0.16 0 -0.68" rpy="0 -0.9 3.14"/>
+  <xacro:wheel name="wheel_front_right" parent="arm_joint_wheel_front_right" xyz="-0.25 0 0" rpy="0 0 0"/>
+  <xacro:arm name="arm_rear_left" parent="base_link" xyz="0.4 0.4 -0.4" rpy="0 -0.9 0"/>
+  <xacro:joint_arm name="arm_joint_wheel_rear_left" parent="arm_rear_left" xyz="0.16 0 -0.68" rpy="0 0.9 0"/>
+  <xacro:wheel name="wheel_rear_left" parent="arm_joint_wheel_rear_left" xyz="0.25 0 0" rpy="0 0 0"/>
+  <xacro:arm name="arm_front_left" parent="base_link" xyz="0.4 -0.38 -0.4" rpy="0 -0.9 0"/>
+  <xacro:joint_arm name="arm_joint_wheel_front_left" parent="arm_front_left" xyz="0.16 0 -0.68" rpy="0 0.9 0"/>
+  <xacro:wheel name="wheel_front_left" parent="arm_joint_wheel_front_left" xyz="0.25 0 0" rpy="0 0 0"/>
+<!--  <ros2_control name="GazeboSystem" type="system">
+    <hardware>
+      <plugin>gazebo_ros2_control/GazeboSystem</plugin>
+    </hardware>
+    <joint name="joint_base_arm_front_left">
+      <command_interface name="position">
+        <param name="min">-0.2</param>
+        <param name="max">0.4</param>
+      </command_interface>
+      <state_interface name="position"/>
+      <state_interface name="velocity"/>
+    </joint>
+    <joint name="joint_base_arm_front_right">
+      <command_interface name="position">
+        <param name="min">-0.2</param>
+        <param name="max">0.4</param>
+      </command_interface>
+      <state_interface name="position"/>
+      <state_interface name="velocity"/>
+    </joint>
+    <joint name="joint_base_arm_rear_left">
+      <command_interface name="position">
+        <param name="min">-0.2</param>
+        <param name="max">0.4</param>
+      </command_interface>
+      <state_interface name="position"/>
+      <state_interface name="velocity"/>
+    </joint>
+    <joint name="joint_base_arm_rear_right">
+      <command_interface name="position">
+        <param name="min">-0.2</param>
+        <param name="max">0.4</param>
+      </command_interface>
+      <state_interface name="position"/>
+      <state_interface name="velocity"/>
+    </joint>
+  </ros2_control>
+  <transmission name="trans_joint_base_arm_front_left">
+    <type>transmission_interface/SimpleTransmission</type>
+    <joint name="joint_base_arm_front_left">
+      <hardwareInterface>PositionJointInterface</hardwareInterface>
+    </joint>
+    <actuator name="motor_arm_front_left">
+      <mechanicalReduction>1.0</mechanicalReduction>
+    </actuator>
+  </transmission>
+  <transmission name="trans_joint_base_arm_front_right">
+    <type>transmission_interface/SimpleTransmission</type>
+    <joint name="joint_base_arm_front_right">
+      <hardwareInterface>PositionJointInterface</hardwareInterface>
+    </joint>
+    <actuator name="motor_arm_front_right">
+      <mechanicalReduction>1.0</mechanicalReduction>
+    </actuator>
+  </transmission>
+  <transmission name="trans_joint_base_arm_rear_left">
+    <type>transmission_interface/SimpleTransmission</type>
+    <joint name="joint_base_arm_rear_left">
+      <hardwareInterface>PositionJointInterface</hardwareInterface>
+    </joint>
+    <actuator name="motor_arm_rear_left">
+      <mechanicalReduction>1.0</mechanicalReduction>
+    </actuator>
+  </transmission>
+  <transmission name="trans_joint_base_arm_rear_right">
+    <type>transmission_interface/SimpleTransmission</type>
+    <joint name="joint_base_arm_rear_right">
+      <hardwareInterface>PositionJointInterface</hardwareInterface>
+    </joint>
+    <actuator name="motor_arm_rear_right">
+      <mechanicalReduction>1.0</mechanicalReduction>
+    </actuator>
+  </transmission>
+  <gazebo>
+    <plugin name="gazebo_ros2_control" filename="libgazebo_ros2_control.so">
+      <robot_param>robot_description</robot_param>
+      <robot_param_node>robot_state_publisher</robot_param_node>
+      <parameters>${controller_config_path}</parameters>
+    </plugin>
+  </gazebo>
+-->
 </robot>

File: urdf/wheel.urdf.xacro (robot description, xacro)
@@ -6,22 +6,23 @@
     <link name="${name}">
       <visual>
-        <origin xyz="0 0 0" rpy="0 0 0"/>
+        <origin xyz="0 0 0" rpy="0 1.57 0"/>
         <geometry>
-          <mesh filename="package://laser_rahcm_visualization/meshes/wheel.dae" scale="0.01 0.01 0.013"/>
+          <mesh filename="package://laser_rahcm_visualization/meshes/wheel.dae" scale="0.008 0.009 0.013"/>
         </geometry>
         <material name="gray"/>
       </visual>
       <collision>
+        <origin xyz="0 0 0" rpy="0 1.57 0"/>
         <geometry>
-          <cylinder radius="0.3" length="0.55"/>
+          <cylinder radius="0.3" length="0.63"/>
         </geometry>
       </collision>
       <inertial>
-        <origin xyz="0 0 0" rpy="0 0 0"/>
-        <mass value="12.5"/>
+        <origin xyz="0 0 0" rpy="0 1.57 0"/>
+        <mass value="3.0"/>
         <inertia
-          ixx="${(1.0/12.0) * 12.5 * (3*(0.3*0.3) + 0.55*0.55)}"
-          iyy="${(1.0/12.0) * 12.5 * (3*(0.3*0.3) + 0.55*0.55)}"
-          izz="${(1.0/2.0) * 12.5 * (0.3*0.3)}"
+          ixx="${(1.0/12.0) * 3.0 * (3*((0.3*0.3)) + 0.63*0.63)}"
+          iyy="${(1.0/2.0) * 3.0 * (0.3*0.3)}"
+          izz="${(1.0/12.0) * 3.0 * (3*((0.3*0.3)) + 0.63*0.63)}"
           ixy="0.0" ixz="0.0" iyz="0.0"/>
       </inertial>
@@ -31,5 +32,5 @@
       <child  link="${name}"/>
       <origin xyz="${xyz}" rpy="${rpy}"/>
-      <axis  xyz="0 0 1"/>
+      <axis  xyz="1 0 0"/>
       <limit  effort="5.0" velocity="10.0"/>
       <dynamics damping="0.1" friction="0.1"/>

File: urdf/wheel_arm_joint.urdf.xacro (robot description, xacro)
@@ -5,4 +5,5 @@
     <link name="${name}">
       <visual>
+        <origin xyz="0 0 0" rpy="0 1.57 0"/>
         <geometry>
           <cylinder length="0.23" radius="0.04"/>
@@ -11,4 +12,5 @@
       </visual>
       <collision>
+        <origin xyz="0 0 0" rpy="0 0 0"/>
         <geometry>
           <cylinder length="0.23" radius="0.04"/>
@@ -16,17 +18,20 @@
       </collision>
       <inertial>
-        <origin xyz="0 0 0" rpy="0 0 0"/>
-        <mass value="2.0"/>
+        <origin xyz="0 0 0" rpy="0 1.57 0"/>
+        <mass value="1.0"/>
         <inertia
-          ixx="${(1.0/12.0) * 2.0 * (3*(0.04*0.04) + 0.23*0.23)}"
-          iyy="${(1.0/12.0) * 2.0 * (3*(0.04*0.04) + 0.23*0.23)}"
-          izz="${(1.0/2.0) * 2.0 * (0.04*0.04)}"
+          ixx="${(1.0/12.0) * 1.0 * (3*(0.04*0.04) + 0.23*0.23)}"
+          iyy="${(1.0/12.0) * 1.0 * (3*(0.04*0.04) + 0.23*0.23)}"
+          izz="${(1.0/2.0) * 1.0 * (0.04*0.04)}"
           ixy="0.0" ixz="0.0" iyz="0.0"/>
       </inertial>
     </link>
-    <joint name="joint_${name}" type="fixed">
+    <joint name="joint_${name}" type="revolute">
       <parent link="${parent}"/>
       <child link="${name}"/>
       <origin xyz="${xyz}" rpy="${rpy}"/>
+      <axis xyz="0 0 0"/>
+      <limit effort="10.0" velocity="1.0" lower="0" upper="0"/>
+      <dynamics damping="5.0" friction="5.0"/>
     </joint>
   </xacro:macro>
