Commit message: implemented thruster plugin

File: urdf/arm.urdf.xacro (robot description, xacro)
@@ -5,11 +5,12 @@
     <link name="${name}">
       <visual>
-        <origin xyz="0 0 -0.3" rpy="0 -0.4 0"/>
+        <origin xyz="0.1 0 -0.6" rpy="0 -0.6 0"/>
         <geometry>
-          <mesh filename="package://laser_rahcm_visualization/meshes/arm.stl" scale="0.01 0.01 0.011"/>
+          <mesh filename="package://laser_rahcm_visualization/meshes/arm.stl" scale="0.01 0.01 0.012"/>
         </geometry>
         <material name="green"/>
       </visual>
       <collision>
+        <origin xyz="0 0 -0.3" rpy="0 -0.4 0"/>
         <geometry>
           <cylinder length="0.55" radius="0.05"/>
@@ -17,17 +18,20 @@
       </collision>
       <inertial>
-        <origin xyz="0 0 0" rpy="0 0 0"/>
+        <origin xyz="0 0 -0.3" rpy="0 -0.4 0"/>
         <mass value="12.5"/>
         <inertia
-          ixx="${(1.0/12.0) * 12.5 * (3*(0.05*0.05) + 0.55*0.55)}"
-          iyy="${(1.0/12.0) * 12.5 * (3*(0.05*0.05) + 0.55*0.55)}"
-          izz="${(1.0/2.0) * 12.5 * (0.05*0.05)}"
+          ixx="${(1.0/2.0) * 3.0 * (0.55*0.55)}"
+          iyy="${(1.0/12.0) * 3.0 * (3*(0.05*0.05) + 0.55*0.55)}"
+          izz="${(1.0/12.0) * 3.0 * (3*(0.05*0.05) + 0.55*0.55)}"
           ixy="0.0" ixz="0.0" iyz="0.0"/>
       </inertial>
     </link>
-    <joint name="joint_${name}" type="fixed">
+    <joint name="joint_base_${name}" type="fixed">
       <parent link="${parent}"/>
       <child link="${name}"/>
       <origin xyz="${xyz}" rpy="${rpy}"/>
+      <axis xyz="0 1 0"/>
+      <limit effort="10.0" velocity="1.0" lower="-0.2" upper="0.4"/>
+      <dynamics damping="5.0" friction="5.0"/>
     </joint>
   </xacro:macro>

File: urdf/base.urdf.xacro (robot description, xacro)
@@ -5,22 +5,23 @@
     <link name="base_link">
       <visual>
-      <origin xyz="0 0 -0.5" rpy="0 0 0"/>
+      <origin xyz="-0.001 0 -0.8" rpy="0 0 0"/>
         <geometry>
-          <mesh filename="package://laser_rahcm_visualization/meshes/chassi.dae" scale="0.0113 0.011 0.0125"/>
+          <mesh filename="package://laser_rahcm_visualization/meshes/chassi.dae" scale="0.0115 0.011 0.0095"/>
         </geometry>
         <material name="white"/>
       </visual>
       <collision>
+        <origin xyz="0 0 -0.5" rpy="0 0 0"/>
         <geometry>
-          <box size="0.8 1.1 0.6"/>
+          <box size="0.71 1.35 0.55"/>
         </geometry>
       </collision>
       <inertial>
-        <origin xyz="0 0 0" rpy="0 0 0"/>
-        <mass value="50"/>
+        <origin xyz="0 0 -0.5" rpy="0 0 0"/>
+        <mass value="50.0"/>
         <inertia
-          ixx="${1.1/12.0 * 50.0 * (0.8*0.8 + 0.6*0.6)}"
-          iyy="${1.1/12.0 * 50.0 * (1.1*1.1 + 0.6*0.6)}"
-          izz="${1.1/12.0 * 50.0 * (0.8*0.8 + 1.1*1.1)}"
+          ixx="${1.0/12.0 * 10.0 * (1.2*1.2 + 0.5*0.5)}"
+          iyy="${1.0/12.0 * 10.0 * (0.8*0.8 + 0.5*0.5)}"
+          izz="${1.0/12.0 * 10.0 * (0.8*0.8 + 1.1*1.1)}"
           ixy="0.0" ixz="0.0" iyz="0.0"/>
       </inertial>

File: urdf/rahcm.urdf.xacro (robot description, xacro)
@@ -19,18 +19,75 @@
     <color rgba="1.0 1.0 1.0 1.0"/>
   </material>
-  <!-- Corpo principal -->
   <xacro:base name="base"/>
-  <!-- Braços e Rodas -->
-  <xacro:arm name="arm_front_left" parent="base_link" xyz="-0.45 0.4 -0.3" rpy="0 -0.9 3.14"/>
-  <xacro:joint_arm name="joint_arm_front_left" parent="arm_front_left" xyz="0 0 -0.35" rpy="0 -0.7 0"/>
-  <xacro:wheel name="wheel_front_left" parent="joint_arm_front_left" xyz="0 0 -0.25" rpy="0 0 0"/>
-  <xacro:arm name="arm_front_right" parent="base_link" xyz="-0.45 -0.38 -0.3" rpy="0 -0.9 3.14"/>
-  <xacro:joint_arm name="joint_arm_front_right" parent="arm_front_right" xyz="0 0 -0.35" rpy="0 -0.7 0"/>
-  <xacro:wheel name="wheel_front_right" parent="joint_arm_front_right" xyz="0 0 -0.25" rpy="0 0 0"/>
-  <xacro:arm name="arm_rear_left" parent="base_link" xyz="0.45 0.4 -0.3" rpy="0 -0.9 0"/>
-  <xacro:joint_arm name="joint_arm_rear_left" parent="arm_rear_left" xyz="0 0 -0.35" rpy="0 -0.7 0"/>
-  <xacro:wheel name="wheel_rear_left" parent="joint_arm_rear_left" xyz="0 0 -0.25" rpy="0 0 0"/>
-  <xacro:arm name="arm_rear_right" parent="base_link" xyz="0.45 -0.38 -0.3" rpy="0 -0.9 0"/>
-  <xacro:joint_arm name="joint_arm_rear_right" parent="arm_rear_right" xyz="0 0 -0.35" rpy="0 -0.7 0"/>
-  <xacro:wheel name="wheel_rear_right" parent="joint_arm_rear_right" xyz="0 0 -0.25" rpy="0 0 0"/>
+  <xacro:arm name="arm_rear_right" parent="base_link" xyz="-0.4 0.4 -0.4" rpy="0 -0.9 3.14"/>
+  <xacro:joint_arm name="arm_joint_wheel_rear_right" parent="arm_rear_right" xyz="0.16 0 -0.68" rpy="0 -0.9 3.14"/>
+  <xacro:wheel name="wheel_rear_right" parent="arm_joint_wheel_rear_right" xyz="-0.25 0 0" rpy="0 0 0"/>
+  <xacro:arm name="arm_front_right" parent="base_link" xyz="-0.4 -0.38 -0.4" rpy="0 -0.9 3.14"/>
+  <xacro:joint_arm name="arm_joint_wheel_front_right" parent="arm_front_right" xyz="0.16 0 -0.68" rpy="0 -0.9 3.14"/>
+  <xacro:wheel name="wheel_front_right" parent="arm_joint_wheel_front_right" xyz="-0.25 0 0" rpy="0 0 0"/>
+  <xacro:arm name="arm_rear_left" parent="base_link" xyz="0.4 0.4 -0.4" rpy="0 -0.9 0"/>
+  <xacro:joint_arm name="arm_joint_wheel_rear_left" parent="arm_rear_left" xyz="0.16 0 -0.68" rpy="0 0.9 0"/>
+  <xacro:wheel name="wheel_rear_left" parent="arm_joint_wheel_rear_left" xyz="0.25 0 0" rpy="0 0 0"/>
+  <xacro:arm name="arm_front_left" parent="base_link" xyz="0.4 -0.38 -0.4" rpy="0 -0.9 0"/>
+  <xacro:joint_arm name="arm_joint_wheel_front_left" parent="arm_front_left" xyz="0.16 0 -0.68" rpy="0 0.9 0"/>
+  <xacro:wheel name="wheel_front_left" parent="arm_joint_wheel_front_left" xyz="0.25 0 0" rpy="0 0 0"/>
+  <gazebo>
+    <plugin name="wamv_gazebo_thrust" filename="libusv_gazebo_thrust_plugin.so">
+        <cmdTimeout>1.0</cmdTimeout>
+        <publisherRate>100.0</publisherRate>
+        <robotNamespace>chico_mendes</robotNamespace>
+        <!-- right front wheel thruster -->
+        <thruster>
+          <linkName>arm_joint_wheel_front_right</linkName>
+          <propJointName>joint_wheel_front_right</propJointName>
+          <engineJointName>joint_joint_arm_front_right</engineJointName>
+          <cmdTopic>thruster/right_front_wheel_cmd</cmdTopic>
+          <angleTopic>right_wheel_angle</angleTopic>
+          <enableAngle>false</enableAngle>
+          <mappingType>1</mappingType>
+          <maxCmd>1.0</maxCmd>
+          <maxForceFwd>1000.0</maxForceFwd>
+          <maxForceRev>-1000.0</maxForceRev>
+        </thruster>
+        <!-- left front wheel thruster -->
+        <thruster>
+          <linkName>arm_joint_wheel_front_left</linkName>
+          <propJointName>joint_wheel_front_left</propJointName>
+          <engineJointName>joint_joint_arm_front_left</engineJointName>
+          <cmdTopic>thruster/left_front_wheel_cmd</cmdTopic>
+          <angleTopic>left_wheel_angle</angleTopic>
+          <enableAngle>false</enableAngle>
+          <mappingType>1</mappingType>
+          <maxCmd>1.0</maxCmd>
+          <maxForceFwd>1000.0</maxForceFwd>
+          <maxForceRev>-1000.0</maxForceRev>
+        </thruster>
+        <!-- right rear wheel thruster -->
+        <thruster>
+          <linkName>arm_joint_wheel_rear_right</linkName>
+          <propJointName>joint_wheel_rear_right</propJointName>
+          <engineJointName>joint_joint_arm_rear_right</engineJointName>
+          <cmdTopic>thruster/right_rear_wheel_cmd</cmdTopic>
+          <angleTopic>right_wheel_angle</angleTopic>
+          <enableAngle>false</enableAngle>
+          <mappingType>1</mappingType>
+          <maxCmd>1.0</maxCmd>
+          <maxForceFwd>1000.0</maxForceFwd>
+          <maxForceRev>-1000.0</maxForceRev>
+        </thruster>
+        <!-- left rear wheel thruster -->
+        <thruster>
+          <linkName>arm_joint_wheel_rear_left</linkName>
+          <propJointName>joint_wheel_rear_left</propJointName>
+          <engineJointName>joint_joint_arm_rear_left</engineJointName>
+          <cmdTopic>thruster/left_rear_wheel_cmd</cmdTopic>
+          <angleTopic>left_wheel_angle</angleTopic>
+          <enableAngle>false</enableAngle>
+          <mappingType>1</mappingType>
+          <maxCmd>1.0</maxCmd>
+          <maxForceFwd>1000.0</maxForceFwd>
+          <maxForceRev>-1000.0</maxForceRev>
+        </thruster>
+    </plugin>
+  </gazebo>
 </robot>

File: urdf/wheel.urdf.xacro (robot description, xacro)
@@ -6,22 +6,23 @@
     <link name="${name}">
       <visual>
-        <origin xyz="0 0 0" rpy="0 0 0"/>
+        <origin xyz="0 0 0" rpy="0 1.57 0"/>
         <geometry>
-          <mesh filename="package://laser_rahcm_visualization/meshes/wheel.dae" scale="0.01 0.01 0.013"/>
+          <mesh filename="package://laser_rahcm_visualization/meshes/wheel.dae" scale="0.008 0.009 0.013"/>
         </geometry>
         <material name="gray"/>
       </visual>
       <collision>
+        <origin xyz="0 0 0" rpy="0 1.57 0"/>
         <geometry>
-          <cylinder radius="0.3" length="0.55"/>
+          <cylinder radius="0.3" length="0.63"/>
         </geometry>
       </collision>
       <inertial>
-        <origin xyz="0 0 0" rpy="0 0 0"/>
+        <origin xyz="0 0 0" rpy="0 1.57 0"/>
         <mass value="12.5"/>
         <inertia
-          ixx="${(1.0/12.0) * 12.5 * (3*(0.3*0.3) + 0.55*0.55)}"
-          iyy="${(1.0/12.0) * 12.5 * (3*(0.3*0.3) + 0.55*0.55)}"
-          izz="${(1.0/2.0) * 12.5 * (0.3*0.3)}"
+          ixx="${(1.0/12.0) * 3.0 * (3*((0.3*0.3)) + 0.63*0.63)}"
+          iyy="${(1.0/2.0) * 3.0 * (0.3*0.3)}"
+          izz="${(1.0/12.0) * 3.0 * (3*((0.3*0.3)) + 0.63*0.63)}"
           ixy="0.0" ixz="0.0" iyz="0.0"/>
       </inertial>
@@ -31,5 +32,5 @@
       <child  link="${name}"/>
       <origin xyz="${xyz}" rpy="${rpy}"/>
-      <axis  xyz="0 0 1"/>
+      <axis  xyz="1 0 0"/>
       <limit  effort="5.0" velocity="10.0"/>
       <dynamics damping="0.1" friction="0.1"/>
@@ -39,5 +40,5 @@
         <bodyName bodyName="${name}"/>
         <!-- Must be same as the ocean model!-->
-        <waterLevel>0.65</waterLevel>
+        <waterLevel>0.9</waterLevel>
         <waterDensity>997.8</waterDensity>
         <!-- Added mass -->
@@ -51,7 +52,7 @@
         <yVV>116.0</yVV>
         <zW>116.0</zW>
-        <kP>10.0</kP>
-        <mQ>10.0</mQ>
-        <nR>10.0</nR>
+        <kP>100.0</kP>
+        <mQ>100.0</mQ>
+        <nR>100.0</nR>
         <nRR>0.0</nRR>
         <!-- General dimensions -->

File: urdf/wheel_arm_joint.urdf.xacro (robot description, xacro)
@@ -5,4 +5,5 @@
     <link name="${name}">
       <visual>
+        <origin xyz="0 0 0" rpy="0 1.57 0"/>
         <geometry>
           <cylinder length="0.23" radius="0.04"/>
@@ -11,4 +12,5 @@
       </visual>
       <collision>
+        <origin xyz="0 0 0" rpy="0 0 0"/>
         <geometry>
           <cylinder length="0.23" radius="0.04"/>
@@ -16,17 +18,20 @@
       </collision>
       <inertial>
-        <origin xyz="0 0 0" rpy="0 0 0"/>
+        <origin xyz="0 0 0" rpy="0 1.57 0"/>
         <mass value="2.0"/>
         <inertia
-          ixx="${(1.0/12.0) * 2.0 * (3*(0.04*0.04) + 0.23*0.23)}"
-          iyy="${(1.0/12.0) * 2.0 * (3*(0.04*0.04) + 0.23*0.23)}"
-          izz="${(1.0/2.0) * 2.0 * (0.04*0.04)}"
+          ixx="${(1.0/12.0) * 1.0 * (3*(0.04*0.04) + 0.23*0.23)}"
+          iyy="${(1.0/12.0) * 1.0 * (3*(0.04*0.04) + 0.23*0.23)}"
+          izz="${(1.0/2.0) * 1.0 * (0.04*0.04)}"
           ixy="0.0" ixz="0.0" iyz="0.0"/>
       </inertial>
     </link>
-    <joint name="joint_${name}" type="fixed">
+    <joint name="joint_${name}" type="revolute">
       <parent link="${parent}"/>
       <child link="${name}"/>
       <origin xyz="${xyz}" rpy="${rpy}"/>
+      <axis xyz="0 0 0"/>
+      <limit effort="10.0" velocity="1.0" lower="0" upper="0"/>
+      <dynamics damping="5.0" friction="5.0"/>
     </joint>
   </xacro:macro>
