Commit message: atualizações feitas no modelo

File: urdf/arm.urdf.xacro (robot description, xacro)
@@ -5,33 +5,30 @@
     <link name="${name}">
       <visual>
-        <origin xyz="0.1 0 -0.6" rpy="0 -0.6 0"/>
+        <origin xyz="0.1 0 -0.6" rpy="0 -0.5 0"/>
         <geometry>
-          <mesh filename="package://laser_rahcm_visualization/meshes/arm.stl" scale="0.01 0.01 0.012"/>
+          <mesh filename="package://laser_rahcm_visualization/meshes/arm.stl" scale="0.01 0.01 0.01"/>
         </geometry>
         <material name="green"/>
       </visual>
       <collision>
-        <origin xyz="0 0 -0.3" rpy="0 -0.4 0"/>
+        <origin xyz="0.05 0 -0.25" rpy="0 0 0.6"/>
         <geometry>
-          <cylinder length="0.55" radius="0.05"/>
+          <cylinder length="0.5" radius="0.05"/>
         </geometry>
       </collision>
       <inertial>
-        <origin xyz="0 0 -0.3" rpy="0 -0.4 0"/>
-        <mass value="3.0"/>
+        <origin xyz="0.05 0 -0.25" rpy="0 0 0.6"/>
+        <mass value="12.5"/>
         <inertia
-          ixx="${(1.0/2.0) * 3.0 * (0.55*0.55)}"
-          iyy="${(1.0/12.0) * 3.0 * (3*(0.05*0.05) + 0.55*0.55)}"
-          izz="${(1.0/12.0) * 3.0 * (3*(0.05*0.05) + 0.55*0.55)}"
+          ixx="${(1.0/12.0) * 12.5 * (3*((0.05*0.05)) + 0.5*0.5)}"
+          iyy="${(1.0/12.0) * 12.5 * (3*((0.05*0.05)) + 0.5*0.5)}"
+          izz="${(1.0/2.0) * 12.5 * ((0.05*0.05))}"
           ixy="0.0" ixz="0.0" iyz="0.0"/>
       </inertial>
     </link>
-    <joint name="joint_base_${name}" type="fixed">
+    <joint name="joint_${name}" type="fixed">
       <parent link="${parent}"/>
       <child link="${name}"/>
       <origin xyz="${xyz}" rpy="${rpy}"/>
-      <axis xyz="0 1 0"/>
-      <limit effort="10.0" velocity="1.0" lower="-0.2" upper="0.4"/>
-      <dynamics damping="5.0" friction="5.0"/>
     </joint>
   </xacro:macro>

File: urdf/base.urdf.xacro (robot description, xacro)
@@ -5,7 +5,7 @@
     <link name="base_link">
       <visual>
-      <origin xyz="-0.001 0 -0.8" rpy="0 0 0"/>
+      <origin xyz="0 0 -0.9" rpy="0 0 1.57"/>
         <geometry>
-          <mesh filename="package://laser_rahcm_visualization/meshes/chassi.dae" scale="0.0115 0.011 0.0095"/>
+          <mesh filename="package://laser_rahcm_visualization/meshes/chassi.dae" scale="0.0113 0.011 0.0125"/>
         </geometry>
         <material name="white"/>
@@ -14,14 +14,14 @@
         <origin xyz="0 0 -0.5" rpy="0 0 0"/>
         <geometry>
-          <box size="0.71 1.35 0.55"/>
+          <box size="1.4 0.7 0.7"/>
         </geometry>
       </collision>
       <inertial>
         <origin xyz="0 0 -0.5" rpy="0 0 0"/>
-        <mass value="10.0"/>
+        <mass value="50"/>
         <inertia
-          ixx="${1.0/12.0 * 10.0 * (1.2*1.2 + 0.5*0.5)}"
-          iyy="${1.0/12.0 * 10.0 * (0.8*0.8 + 0.5*0.5)}"
-          izz="${1.0/12.0 * 10.0 * (0.8*0.8 + 1.1*1.1)}"
+          ixx="${(1.0/12.0) * 50.0 * ((1.4*1.4) + (0.7*0.7))}"
+          iyy="${(1.0/12.0) * 50.0 * ((0.7*0.7) + (0.7*0.7))}"
+          izz="${(1.0/12.0) * 50.0 * ((0.7*0.7) + (1.4*1.4))}"
           ixy="0.0" ixz="0.0" iyz="0.0"/>
       </inertial>

File: urdf/rahcm.urdf.xacro (robot description, xacro)
@@ -21,96 +21,15 @@
   </material>
   <xacro:base name="base"/>
-  <xacro:arm name="arm_rear_right" parent="base_link" xyz="-0.4 0.4 -0.4" rpy="0 -0.9 3.14"/>
-  <xacro:joint_arm name="arm_joint_wheel_rear_right" parent="arm_rear_right" xyz="0.16 0 -0.68" rpy="0 -0.9 3.14"/>
-  <xacro:wheel name="wheel_rear_right" parent="arm_joint_wheel_rear_right" xyz="-0.25 0 0" rpy="0 0 0"/>
-  <xacro:arm name="arm_front_right" parent="base_link" xyz="-0.4 -0.38 -0.4" rpy="0 -0.9 3.14"/>
-  <xacro:joint_arm name="arm_joint_wheel_front_right" parent="arm_front_right" xyz="0.16 0 -0.68" rpy="0 -0.9 3.14"/>
-  <xacro:wheel name="wheel_front_right" parent="arm_joint_wheel_front_right" xyz="-0.25 0 0" rpy="0 0 0"/>
-  <xacro:arm name="arm_rear_left" parent="base_link" xyz="0.4 0.4 -0.4" rpy="0 -0.9 0"/>
-  <xacro:joint_arm name="arm_joint_wheel_rear_left" parent="arm_rear_left" xyz="0.16 0 -0.68" rpy="0 0.9 0"/>
-  <xacro:wheel name="wheel_rear_left" parent="arm_joint_wheel_rear_left" xyz="0.25 0 0" rpy="0 0 0"/>
-  <xacro:arm name="arm_front_left" parent="base_link" xyz="0.4 -0.38 -0.4" rpy="0 -0.9 0"/>
-  <xacro:joint_arm name="arm_joint_wheel_front_left" parent="arm_front_left" xyz="0.16 0 -0.68" rpy="0 0.9 0"/>
-  <xacro:wheel name="wheel_front_left" parent="arm_joint_wheel_front_left" xyz="0.25 0 0" rpy="0 0 0"/>
-<!--  <ros2_control name="GazeboSystem" type="system">
-    <hardware>
-      <plugin>gazebo_ros2_control/GazeboSystem</plugin>
-    </hardware>
-    <joint name="joint_base_arm_front_left">
-      <command_interface name="position">
-        <param name="min">-0.2</param>
-        <param name="max">0.4</param>
-      </command_interface>
-      <state_interface name="position"/>
-      <state_interface name="velocity"/>
-    </joint>
-    <joint name="joint_base_arm_front_right">
-      <command_interface name="position">
-        <param name="min">-0.2</param>
-        <param name="max">0.4</param>
-      </command_interface>
-      <state_interface name="position"/>
-      <state_interface name="velocity"/>
-    </joint>
-    <joint name="joint_base_arm_rear_left">
-      <command_interface name="position">
-        <param name="min">-0.2</param>
-        <param name="max">0.4</param>
-      </command_interface>
-      <state_interface name="position"/>
-      <state_interface name="velocity"/>
-    </joint>
-    <joint name="joint_base_arm_rear_right">
-      <command_interface name="position">
-        <param name="min">-0.2</param>
-        <param name="max">0.4</param>
-      </command_interface>
-      <state_interface name="position"/>
-      <state_interface name="velocity"/>
-    </joint>
-  </ros2_control>
-  <transmission name="trans_joint_base_arm_front_left">
-    <type>transmission_interface/SimpleTransmission</type>
-    <joint name="joint_base_arm_front_left">
-      <hardwareInterface>PositionJointInterface</hardwareInterface>
-    </joint>
-    <actuator name="motor_arm_front_left">
-      <mechanicalReduction>1.0</mechanicalReduction>
-    </actuator>
-  </transmission>
-  <transmission name="trans_joint_base_arm_front_right">
-    <type>transmission_interface/SimpleTransmission</type>
-    <joint name="joint_base_arm_front_right">
-      <hardwareInterface>PositionJointInterface</hardwareInterface>
-    </joint>
-    <actuator name="motor_arm_front_right">
-      <mechanicalReduction>1.0</mechanicalReduction>
-    </actuator>
-  </transmission>
-  <transmission name="trans_joint_base_arm_rear_left">
-    <type>transmission_interface/SimpleTransmission</type>
-    <joint name="joint_base_arm_rear_left">
-      <hardwareInterface>PositionJointInterface</hardwareInterface>
-    </joint>
-    <actuator name="motor_arm_rear_left">
-      <mechanicalReduction>1.0</mechanicalReduction>
-    </actuator>
-  </transmission>
-  <transmission name="trans_joint_base_arm_rear_right">
-    <type>transmission_interface/SimpleTransmission</type>
-    <joint name="joint_base_arm_rear_right">
-      <hardwareInterface>PositionJointInterface</hardwareInterface>
-    </joint>
-    <actuator name="motor_arm_rear_right">
-      <mechanicalReduction>1.0</mechanicalReduction>
-    </actuator>
-  </transmission>
-  <gazebo>
-    <plugin name="gazebo_ros2_control" filename="libgazebo_ros2_control.so">
-      <robot_param>robot_description</robot_param>
-      <robot_param_node>robot_state_publisher</robot_param_node>
-      <parameters>${controller_config_path}</parameters>
-    </plugin>
-  </gazebo>
--->
+  <xacro:arm name="arm_rear_left" parent="base_link" xyz="-0.4 0.2 -0.5" rpy="0 -0.8 1.5708"/>
+  <xacro:joint_arm name="arm_joint_wheel_rear_left" parent="arm_rear_left" xyz="0.16 0 -0.68" rpy="-0.80165 0 -1.5708"/>
+  <xacro:wheel name="wheel_rear_left" parent="arm_joint_wheel_rear_left" xyz="0 0.25 0" rpy="0 0 0"/>
+  <xacro:arm name="arm_rear_right" parent="base_link" xyz="-0.4 -0.2 -0.5" rpy="0 -0.8 -1.57"/>
+  <xacro:joint_arm name="arm_joint_wheel_rear_right" parent="arm_rear_right" xyz="0.16 0 -0.68" rpy="-0.80165 0 -1.5708"/>
+  <xacro:wheel name="wheel_rear_right" parent="arm_joint_wheel_rear_right" xyz="0 0.25 0" rpy="0 0 0"/>
+  <xacro:arm name="arm_front_left" parent="base_link" xyz="0.4 0.2 -0.5" rpy="0 -0.8 1.5708"/>
+  <xacro:joint_arm name="arm_joint_wheel_front_left" parent="arm_front_left" xyz="0.16 0 -0.68" rpy="-0.80165 0 -1.5708"/>
+  <xacro:wheel name="wheel_front_left" parent="arm_joint_wheel_front_left" xyz="0 0.25 0" rpy="0 0 0"/>
+  <xacro:arm name="arm_front_right" parent="base_link" xyz="0.4 -0.2 -0.5" rpy="0 -0.8 -1.5708"/>
+  <xacro:joint_arm name="arm_joint_wheel_front_right" parent="arm_front_right" xyz="0.16 0 -0.68" rpy="-0.80165 0 -1.5708"/>
+  <xacro:wheel name="wheel_front_right" parent="arm_joint_wheel_front_right" xyz="0 0.25 0" rpy="0 0 0"/>
 </robot>

File: urdf/wheel.urdf.xacro (robot description, xacro)
@@ -6,23 +6,23 @@
     <link name="${name}">
       <visual>
-        <origin xyz="0 0 0" rpy="0 1.57 0"/>
+        <origin xyz="0 0 0" rpy="1.5708 0 0"/>
         <geometry>
-          <mesh filename="package://laser_rahcm_visualization/meshes/wheel.dae" scale="0.008 0.009 0.013"/>
+          <mesh filename="package://laser_rahcm_visualization/meshes/wheel.dae" scale="0.0093 0.0093 0.013"/>
         </geometry>
         <material name="gray"/>
       </visual>
       <collision>
-        <origin xyz="0 0 0" rpy="0 1.57 0"/>
+        <origin xyz="0 0.03 0" rpy="1.5708 0 0"/>
         <geometry>
-          <cylinder radius="0.3" length="0.63"/>
+          <cylinder radius="0.3" length="0.6"/>
         </geometry>
       </collision>
       <inertial>
-        <origin xyz="0 0 0" rpy="0 1.57 0"/>
-        <mass value="3.0"/>
+        <origin xyz="0 0.03 0" rpy="1.5708 0 0"/>
+        <mass value="12.5"/>
         <inertia
-          ixx="${(1.0/12.0) * 3.0 * (3*((0.3*0.3)) + 0.63*0.63)}"
-          iyy="${(1.0/2.0) * 3.0 * (0.3*0.3)}"
-          izz="${(1.0/12.0) * 3.0 * (3*((0.3*0.3)) + 0.63*0.63)}"
+          ixx="${(1.0/12.0) * 12.5 * (3*(0.3*0.3) + 0.6*0.6)}"
+          iyy="${(1.0/12.0) * 12.5 * (3*(0.3*0.3) + 0.6*0.6)}"
+          izz="${(1.0/2.0) * 12.5 * (0.3*0.3)}"
           ixy="0.0" ixz="0.0" iyz="0.0"/>
       </inertial>
@@ -32,5 +32,5 @@
       <child  link="${name}"/>
       <origin xyz="${xyz}" rpy="${rpy}"/>
-      <axis  xyz="1 0 0"/>
+      <axis  xyz="0 1.5708 0"/>
       <limit  effort="5.0" velocity="10.0"/>
       <dynamics damping="0.1" friction="0.1"/>
@@ -40,5 +40,5 @@
         <bodyName bodyName="${name}"/>
         <!-- Must be same as the ocean model!-->
-        <waterLevel>0.65</waterLevel>
+        <waterLevel>0.9</waterLevel>
         <waterDensity>997.8</waterDensity>
         <!-- Added mass -->

File: urdf/wheel_arm_joint.urdf.xacro (robot description, xacro)
@@ -5,5 +5,5 @@
     <link name="${name}">
       <visual>
-        <origin xyz="0 0 0" rpy="0 1.57 0"/>
+        <origin xyz="0 0 0" rpy="1.5708 0 0"/>
         <geometry>
           <cylinder length="0.23" radius="0.04"/>
@@ -12,5 +12,5 @@
       </visual>
       <collision>
-        <origin xyz="0 0 0" rpy="0 0 0"/>
+        <origin xyz="0 0 0" rpy="1.5708 0 0"/>
         <geometry>
           <cylinder length="0.23" radius="0.04"/>
@@ -18,10 +18,10 @@
       </collision>
       <inertial>
-        <origin xyz="0 0 0" rpy="0 1.57 0"/>
-        <mass value="1.0"/>
+        <origin xyz="0 0 0" rpy="1.5708 0 0"/>
+        <mass value="2.0"/>
         <inertia
-          ixx="${(1.0/12.0) * 1.0 * (3*(0.04*0.04) + 0.23*0.23)}"
-          iyy="${(1.0/12.0) * 1.0 * (3*(0.04*0.04) + 0.23*0.23)}"
-          izz="${(1.0/2.0) * 1.0 * (0.04*0.04)}"
+          ixx="${(1.0/12.0) * 2.0 * (3*(0.04*0.04) + 0.23*0.23)}"
+          iyy="${(1.0/12.0) * 2.0 * (3*(0.04*0.04) + 0.23*0.23)}"
+          izz="${(1.0/2.0) * 2.0 * (0.04*0.04)}"
           ixy="0.0" ixz="0.0" iyz="0.0"/>
       </inertial>
@@ -31,5 +31,5 @@
       <child link="${name}"/>
       <origin xyz="${xyz}" rpy="${rpy}"/>
-      <axis xyz="0 0 0"/>
+      <axis xyz="1 0 0"/>
       <limit effort="10.0" velocity="1.0" lower="0" upper="0"/>
       <dynamics damping="5.0" friction="5.0"/>
