Commit message: link das rodas

File: urdf/base.urdf.xacro (robot description, xacro)
@@ -12,14 +12,14 @@
       <collision>
         <geometry>
-          <box size="0.8 1 0.6"/>
+          <box size="0.8 1.5 0.6"/>
         </geometry>
       </collision>
       <inertial>
         <origin xyz="0 0 0.3" rpy="0 0 0"/>
-        <mass value="80"/>
+        <mass value="60"/>
         <inertia
-          ixx="${1.5/12.0 * 80.0 * (0.8*0.8 + 0.6*0.6)}"
-          iyy="${1.5/12.0 * 80.0 * (1.5*1.5 + 0.6*0.6)}"
-          izz="${1.5/12.0 * 80.0 * (0.8*0.8 + 1.5*1.5)}"
+          ixx="${1.5/12.0 * 60.0 * (0.8*0.8 + 0.6*0.6)}"
+          iyy="${1.5/12.0 * 60.0 * (1.5*1.5 + 0.6*0.6)}"
+          izz="${1.5/12.0 * 60.0 * (0.8*0.8 + 1.5*1.5)}"
           ixy="0.0" ixz="0.0" iyz="0.0"/>
       </inertial>

File: urdf/wheel.urdf.xacro (robot description, xacro)
@@ -17,16 +17,19 @@
       <inertial>
         <origin xyz="0 0 0" rpy="0 0 0"/>
-        <mass value="5"/>
+        <mass value="10"/>
         <inertia
-          ixx="${(2/5) * 5.0 * (0.3*0.3)}"
-          iyy="${(2/5) * 5.0 * (0.3*0.3)}"
-          izz="${(2/5) * 5.0 * (0.3*0.3)}"
+          ixx="${(2/5) * 10.0 * (0.3*0.3)}"
+          iyy="${(2/5) * 10.0 * (0.3*0.3)}"
+          izz="${(2/5) * 10.0 * (0.3*0.3)}"
           ixy="0.0" ixz="0.0" iyz="0.0"/>
       </inertial>
     </link>
-    <joint name="joint_${name}" type="fixed">
+    <joint name="joint_${name}" type="revolute">
       <parent link="${parent}"/>
       <child link="${name}"/>
       <origin xyz="${xyz}" rpy="${rpy}"/>
+      <axis xyz="1 0 0"/>
+      <limit effort="5.0" velocity="10.0"/>
+      <dynamics damping="0.1" friction="0.1"/>
     </joint>
   </xacro:macro>

Commit message: mudança no link do pino

File: urdf/base.urdf.xacro (robot description, xacro)
@@ -5,5 +5,5 @@
     <link name="base_link">
       <visual>
-      <origin xyz="0 0 -0.9" rpy="0 0 1.57"/>
+      <origin xyz="0 0 -0.75" rpy="0 0 1.57"/>
         <geometry>
           <mesh filename="package://laser_rahcm_visualization/meshes/chassi.dae" scale="0.0113 0.011 0.0125"/>

File: urdf/rahcm.urdf.xacro (robot description, xacro)
@@ -21,15 +21,15 @@
   </material>
   <xacro:base name="base"/>
-  <xacro:arm name="arm_rear_left" parent="base_link" xyz="-0.4 0.2 -0.5" rpy="0 -0.8 1.5708"/>
+  <xacro:arm name="arm_rear_left" parent="base_link" xyz="-0.4 0.2 -0.4" rpy="0 -0.8 1.5708"/>
   <xacro:joint_arm name="arm_joint_wheel_rear_left" parent="arm_rear_left" xyz="0.16 0 -0.68" rpy="-0.80165 0 -1.5708"/>
   <xacro:wheel name="wheel_rear_left" parent="arm_joint_wheel_rear_left" xyz="0 0.25 0" rpy="0 0 0"/>
-  <xacro:arm name="arm_rear_right" parent="base_link" xyz="-0.4 -0.2 -0.5" rpy="0 -0.8 -1.57"/>
-  <xacro:joint_arm name="arm_joint_wheel_rear_right" parent="arm_rear_right" xyz="0.16 0 -0.68" rpy="-0.80165 0 -1.5708"/>
-  <xacro:wheel name="wheel_rear_right" parent="arm_joint_wheel_rear_right" xyz="0 0.25 0" rpy="0 0 0"/>
-  <xacro:arm name="arm_front_left" parent="base_link" xyz="0.4 0.2 -0.5" rpy="0 -0.8 1.5708"/>
+  <xacro:arm name="arm_rear_right" parent="base_link" xyz="-0.4 -0.2 -0.4" rpy="0 -0.8 -1.57"/>
+  <xacro:joint_arm name="arm_joint_wheel_rear_right" parent="arm_rear_right" xyz="0.16 0 -0.68" rpy="0.80165 0 1.5708"/>
+  <xacro:wheel name="wheel_rear_right" parent="arm_joint_wheel_rear_right" xyz="0 -0.25 0" rpy="0 0 3.14159"/>
+  <xacro:arm name="arm_front_left" parent="base_link" xyz="0.4 0.2 -0.4" rpy="0 -0.8 1.5708"/>
   <xacro:joint_arm name="arm_joint_wheel_front_left" parent="arm_front_left" xyz="0.16 0 -0.68" rpy="-0.80165 0 -1.5708"/>
   <xacro:wheel name="wheel_front_left" parent="arm_joint_wheel_front_left" xyz="0 0.25 0" rpy="0 0 0"/>
-  <xacro:arm name="arm_front_right" parent="base_link" xyz="0.4 -0.2 -0.5" rpy="0 -0.8 -1.5708"/>
-  <xacro:joint_arm name="arm_joint_wheel_front_right" parent="arm_front_right" xyz="0.16 0 -0.68" rpy="-0.80165 0 -1.5708"/>
-  <xacro:wheel name="wheel_front_right" parent="arm_joint_wheel_front_right" xyz="0 0.25 0" rpy="0 0 0"/>
+  <xacro:arm name="arm_front_right" parent="base_link" xyz="0.4 -0.2 -0.4" rpy="0 -0.8 -1.5708"/>
+  <xacro:joint_arm name="arm_joint_wheel_front_right" parent="arm_front_right" xyz="0.16 0 -0.68" rpy="0.80165 0 1.5708"/>
+  <xacro:wheel name="wheel_front_right" parent="arm_joint_wheel_front_right" xyz="0 -0.25 0" rpy="0 0 3.14159"/>
 </robot>

Commit message: fixed robot frames and adjusted thruster plugin

File: urdf/base.urdf.xacro (robot description, xacro)
@@ -5,7 +5,7 @@
     <link name="base_link">
       <visual>
-      <origin xyz="-0.001 0 -0.8" rpy="0 0 0"/>
+      <origin xyz="0 0 -0.75" rpy="0 0 1.57"/>
         <geometry>
-          <mesh filename="package://laser_rahcm_visualization/meshes/chassi.dae" scale="0.0115 0.011 0.0095"/>
+          <mesh filename="package://laser_rahcm_visualization/meshes/chassi.dae" scale="0.0113 0.011 0.0125"/>
         </geometry>
         <material name="white"/>
@@ -14,14 +14,14 @@
         <origin xyz="0 0 -0.5" rpy="0 0 0"/>
         <geometry>
-          <box size="0.71 1.35 0.55"/>
+          <box size="1.4 0.7 0.7"/>
         </geometry>
       </collision>
       <inertial>
         <origin xyz="0 0 -0.5" rpy="0 0 0"/>
-        <mass value="50.0"/>
+        <mass value="50"/>
         <inertia
-          ixx="${1.0/12.0 * 10.0 * (1.2*1.2 + 0.5*0.5)}"
-          iyy="${1.0/12.0 * 10.0 * (0.8*0.8 + 0.5*0.5)}"
-          izz="${1.0/12.0 * 10.0 * (0.8*0.8 + 1.1*1.1)}"
+          ixx="${(1.0/12.0) * 50.0 * ((1.4*1.4) + (0.7*0.7))}"
+          iyy="${(1.0/12.0) * 50.0 * ((0.7*0.7) + (0.7*0.7))}"
+          izz="${(1.0/12.0) * 50.0 * ((0.7*0.7) + (1.4*1.4))}"
           ixy="0.0" ixz="0.0" iyz="0.0"/>
       </inertial>

File: urdf/rahcm.urdf.xacro (robot description, xacro)
@@ -1,9 +1,8 @@
 <?xml version="1.0"?>
 <robot name="laser_rahcm_visualization" xmlns:xacro="http://ros.org/wiki/xacro">
-  <!-- Importa os módulos -->
   <xacro:include filename="base.urdf.xacro"/>
   <xacro:include filename="arm.urdf.xacro"/>
+  <xacro:include filename="wheel_arm_joint.urdf.xacro"/>
   <xacro:include filename="wheel.urdf.xacro"/>
-  <xacro:include filename="wheel_arm_joint.urdf.xacro"/>
   <!-- Define materiais -->
   <material name="gray">
@@ -20,16 +19,16 @@
   </material>
   <xacro:base name="base"/>
-  <xacro:arm name="arm_rear_right" parent="base_link" xyz="-0.4 0.4 -0.4" rpy="0 -0.9 3.14"/>
-  <xacro:joint_arm name="arm_joint_wheel_rear_right" parent="arm_rear_right" xyz="0.16 0 -0.68" rpy="0 -0.9 3.14"/>
-  <xacro:wheel name="wheel_rear_right" parent="arm_joint_wheel_rear_right" xyz="-0.25 0 0" rpy="0 0 0"/>
-  <xacro:arm name="arm_front_right" parent="base_link" xyz="-0.4 -0.38 -0.4" rpy="0 -0.9 3.14"/>
-  <xacro:joint_arm name="arm_joint_wheel_front_right" parent="arm_front_right" xyz="0.16 0 -0.68" rpy="0 -0.9 3.14"/>
-  <xacro:wheel name="wheel_front_right" parent="arm_joint_wheel_front_right" xyz="-0.25 0 0" rpy="0 0 0"/>
-  <xacro:arm name="arm_rear_left" parent="base_link" xyz="0.4 0.4 -0.4" rpy="0 -0.9 0"/>
-  <xacro:joint_arm name="arm_joint_wheel_rear_left" parent="arm_rear_left" xyz="0.16 0 -0.68" rpy="0 0.9 0"/>
-  <xacro:wheel name="wheel_rear_left" parent="arm_joint_wheel_rear_left" xyz="0.25 0 0" rpy="0 0 0"/>
-  <xacro:arm name="arm_front_left" parent="base_link" xyz="0.4 -0.38 -0.4" rpy="0 -0.9 0"/>
-  <xacro:joint_arm name="arm_joint_wheel_front_left" parent="arm_front_left" xyz="0.16 0 -0.68" rpy="0 0.9 0"/>
-  <xacro:wheel name="wheel_front_left" parent="arm_joint_wheel_front_left" xyz="0.25 0 0" rpy="0 0 0"/>
+  <xacro:arm name="arm_rear_left" parent="base_link" xyz="-0.4 0.2 -0.4" rpy="0 -0.8 1.5708"/>
+  <xacro:joint_arm name="arm_joint_wheel_rear_left" parent="arm_rear_left" xyz="0.16 0 -0.68" rpy="-0.80165 0 -1.5708"/>
+  <xacro:wheel name="wheel_rear_left" parent="arm_joint_wheel_rear_left" xyz="0 0.25 0" rpy="0 0 0"/>
+  <xacro:arm name="arm_rear_right" parent="base_link" xyz="-0.4 -0.2 -0.4" rpy="0 -0.8 -1.57"/>
+  <xacro:joint_arm name="arm_joint_wheel_rear_right" parent="arm_rear_right" xyz="0.16 0 -0.68" rpy="0.80165 0 1.5708"/>
+  <xacro:wheel name="wheel_rear_right" parent="arm_joint_wheel_rear_right" xyz="0 -0.25 0" rpy="0 0 3.14159"/>
+  <xacro:arm name="arm_front_left" parent="base_link" xyz="0.4 0.2 -0.4" rpy="0 -0.8 1.5708"/>
+  <xacro:joint_arm name="arm_joint_wheel_front_left" parent="arm_front_left" xyz="0.16 0 -0.68" rpy="-0.80165 0 -1.5708"/>
+  <xacro:wheel name="wheel_front_left" parent="arm_joint_wheel_front_left" xyz="0 0.25 0" rpy="0 0 0"/>
+  <xacro:arm name="arm_front_right" parent="base_link" xyz="0.4 -0.2 -0.4" rpy="0 -0.8 -1.5708"/>
+  <xacro:joint_arm name="arm_joint_wheel_front_right" parent="arm_front_right" xyz="0.16 0 -0.68" rpy="0.80165 0 1.5708"/>
+  <xacro:wheel name="wheel_front_right" parent="arm_joint_wheel_front_right" xyz="0 -0.25 0" rpy="0 0 3.14159"/>
   <gazebo>
     <plugin name="wamv_gazebo_thrust" filename="libusv_gazebo_thrust_plugin.so">
@@ -45,8 +44,8 @@
           <angleTopic>right_wheel_angle</angleTopic>
           <enableAngle>false</enableAngle>
-          <mappingType>1</mappingType>
+          <mappingType>0</mappingType>
           <maxCmd>1.0</maxCmd>
-          <maxForceFwd>1000.0</maxForceFwd>
-          <maxForceRev>-1000.0</maxForceRev>
+          <maxForceFwd>500.0</maxForceFwd>
+          <maxForceRev>-250.0</maxForceRev>
         </thruster>
         <!-- left front wheel thruster -->
@@ -58,8 +57,8 @@
           <angleTopic>left_wheel_angle</angleTopic>
           <enableAngle>false</enableAngle>
-          <mappingType>1</mappingType>
+          <mappingType>0</mappingType>
           <maxCmd>1.0</maxCmd>
-          <maxForceFwd>1000.0</maxForceFwd>
-          <maxForceRev>-1000.0</maxForceRev>
+          <maxForceFwd>500.0</maxForceFwd>
+          <maxForceRev>-250.0</maxForceRev>
         </thruster>
         <!-- right rear wheel thruster -->
@@ -71,8 +70,8 @@
           <angleTopic>right_wheel_angle</angleTopic>
           <enableAngle>false</enableAngle>
-          <mappingType>1</mappingType>
+          <mappingType>0</mappingType>
           <maxCmd>1.0</maxCmd>
-          <maxForceFwd>1000.0</maxForceFwd>
-          <maxForceRev>-1000.0</maxForceRev>
+          <maxForceFwd>500.0</maxForceFwd>
+          <maxForceRev>-250.0</maxForceRev>
         </thruster>
         <!-- left rear wheel thruster -->
@@ -84,8 +83,8 @@
           <angleTopic>left_wheel_angle</angleTopic>
           <enableAngle>false</enableAngle>
-          <mappingType>1</mappingType>
+          <mappingType>0</mappingType>
           <maxCmd>1.0</maxCmd>
-          <maxForceFwd>1000.0</maxForceFwd>
-          <maxForceRev>-1000.0</maxForceRev>
+          <maxForceFwd>500.0</maxForceFwd>
+          <maxForceRev>-250.0</maxForceRev>
         </thruster>
     </plugin>

File: urdf/wheel.urdf.xacro (robot description, xacro)
@@ -6,23 +6,23 @@
     <link name="${name}">
       <visual>
-        <origin xyz="0 0 0" rpy="0 1.57 0"/>
+        <origin xyz="0 0 0" rpy="1.5708 0 0"/>
         <geometry>
-          <mesh filename="package://laser_rahcm_visualization/meshes/wheel.dae" scale="0.008 0.009 0.013"/>
+          <mesh filename="package://laser_rahcm_visualization/meshes/wheel.dae" scale="0.0093 0.0093 0.013"/>
         </geometry>
         <material name="gray"/>
       </visual>
       <collision>
-        <origin xyz="0 0 0" rpy="0 1.57 0"/>
+        <origin xyz="0 0.03 0" rpy="1.5708 0 0"/>
         <geometry>
-          <cylinder radius="0.3" length="0.63"/>
+          <cylinder radius="0.3" length="0.6"/>
         </geometry>
       </collision>
       <inertial>
-        <origin xyz="0 0 0" rpy="0 1.57 0"/>
+        <origin xyz="0 0.03 0" rpy="1.5708 0 0"/>
         <mass value="12.5"/>
         <inertia
-          ixx="${(1.0/12.0) * 3.0 * (3*((0.3*0.3)) + 0.63*0.63)}"
-          iyy="${(1.0/2.0) * 3.0 * (0.3*0.3)}"
-          izz="${(1.0/12.0) * 3.0 * (3*((0.3*0.3)) + 0.63*0.63)}"
+          ixx="${(1.0/12.0) * 12.5 * (3*(0.3*0.3) + 0.6*0.6)}"
+          iyy="${(1.0/12.0) * 12.5 * (3*(0.3*0.3) + 0.6*0.6)}"
+          izz="${(1.0/2.0) * 12.5 * (0.3*0.3)}"
           ixy="0.0" ixz="0.0" iyz="0.0"/>
       </inertial>
@@ -32,5 +32,5 @@
       <child  link="${name}"/>
       <origin xyz="${xyz}" rpy="${rpy}"/>
-      <axis  xyz="1 0 0"/>
+      <axis  xyz="0 1.5708 0"/>
       <limit  effort="5.0" velocity="10.0"/>
       <dynamics damping="0.1" friction="0.1"/>

File: urdf/wheel_arm_joint.urdf.xacro (robot description, xacro)
@@ -5,5 +5,5 @@
     <link name="${name}">
       <visual>
-        <origin xyz="0 0 0" rpy="0 1.57 0"/>
+        <origin xyz="0 0 0" rpy="1.5708 0 0"/>
         <geometry>
           <cylinder length="0.23" radius="0.04"/>
@@ -12,5 +12,5 @@
       </visual>
       <collision>
-        <origin xyz="0 0 0" rpy="0 0 0"/>
+        <origin xyz="0 0 0" rpy="1.5708 0 0"/>
         <geometry>
           <cylinder length="0.23" radius="0.04"/>
@@ -18,10 +18,10 @@
       </collision>
       <inertial>
-        <origin xyz="0 0 0" rpy="0 1.57 0"/>
+        <origin xyz="0 0 0" rpy="1.5708 0 0"/>
         <mass value="2.0"/>
         <inertia
-          ixx="${(1.0/12.0) * 1.0 * (3*(0.04*0.04) + 0.23*0.23)}"
-          iyy="${(1.0/12.0) * 1.0 * (3*(0.04*0.04) + 0.23*0.23)}"
-          izz="${(1.0/2.0) * 1.0 * (0.04*0.04)}"
+          ixx="${(1.0/12.0) * 2.0 * (3*(0.04*0.04) + 0.23*0.23)}"
+          iyy="${(1.0/12.0) * 2.0 * (3*(0.04*0.04) + 0.23*0.23)}"
+          izz="${(1.0/2.0) * 2.0 * (0.04*0.04)}"
           ixy="0.0" ixz="0.0" iyz="0.0"/>
       </inertial>
@@ -31,5 +31,5 @@
       <child link="${name}"/>
       <origin xyz="${xyz}" rpy="${rpy}"/>
-      <axis xyz="0 0 0"/>
+      <axis xyz="1 0 0"/>
       <limit effort="10.0" velocity="1.0" lower="0" upper="0"/>
       <dynamics damping="5.0" friction="5.0"/>
